Commit message: added desired_state

File: simulation/urdf/ground.urdf (robot description, URDF)
Before this commit: robot ground_skeleton, 2 links, 1 joints
Links:
- link ground_link: geometry collision box size=11.5 0.05 11.5; visual box size=0.5 0.0501 0.5
Joints:
- joint ground_joint: origin xyz=0 0 0 rpy=0 0 0 -> xyz=0 0 -0.025 rpy=0 0 0

File: simulation/urdf/hrp4/urdf/hrp4.urdf (robot description, URDF)
Before this commit: robot hrp4, 66 links, 65 joints
Links:
- removed link Accelerometer
- removed link Gyro
- removed link LeftFootForceSensor
- removed link LeftHandForceSensor
- removed link RightFootForceSensor
- removed link RightHandForceSensor
- removed link base_link
- removed link gaze
- removed link l_gripper
- removed link r_gripper
- removed link r_gripper_sensor
- link l_sole: mass 0.0001 -> 0.001
- link r_sole: mass 1 -> 0.001
Joints:
- removed joint AccelerometerJoint
- removed joint GyroJoint
- removed joint LeftFootForceSensorJoint
- removed joint LeftHandForceSensorJoint
- removed joint RightFootForceSensorJoint
- removed joint RightHandForceSensorJoint
- removed joint gaze_joint
- removed joint l_gripper_joint
- removed joint r_gripper_joint
- removed joint r_gripper_sensor
- removed joint waist
- joint L_F22: type revolute -> fixed
- joint L_F23: type revolute -> fixed
- joint L_F32: type revolute -> fixed
- joint L_F33: type revolute -> fixed
- joint L_F42: type revolute -> fixed
- joint L_F43: type revolute -> fixed
- joint L_F52: type revolute -> fixed
- joint L_F53: type revolute -> fixed
- joint L_HAND_J0: type revolute -> fixed
- joint L_HAND_J1: type revolute -> fixed
- joint L_WRIST_P: type revolute -> fixed
- joint L_WRIST_R: type revolute -> fixed
- joint L_WRIST_Y: type revolute -> fixed
- joint R_F22: type revolute -> fixed
- joint R_F23: type revolute -> fixed
- joint R_F32: type revolute -> fixed
- joint R_F33: type revolute -> fixed
- joint R_F42: type revolute -> fixed
- joint R_F43: type revolute -> fixed
- joint R_F52: type revolute -> fixed
- joint R_F53: type revolute -> fixed
- joint R_HAND_J0: type revolute -> fixed
- joint R_HAND_J1: type revolute -> fixed
- joint R_WRIST_P: type revolute -> fixed
- joint R_WRIST_R: type revolute -> fixed
- joint R_WRIST_Y: type revolute -> fixed
