Commit message: qp is more general now: you can select to have the whole lip state and zmp velocity as decision variable, or just the zmp position and zmp velocity as decision variable

File: simulation/models/nao/urdf/nao.urdf (robot description, URDF)
Before this commit: robot NaoH25V50, 30 links, 29 joints
Links:
- link LSole: mass None -> 0.001
- link RSole: mass None -> 0.001
